File: Coil.kicad_sch (KiCad schematic)
At the start: 54 parts, among them Q400 STL20N6F7, Q401 STL20N6F7, Q402 STL20N6F7, Q403 STL20N6F7, Q406 STL20N6F7, Q407 STL20N6F7, Q408 STL20N6F7, Q409 STL20N6F7, Q410 NPN, Q411 BC856BMTF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

Commit message: PCB Layout V1.1
Parts:
- renumbered R402 to R403, R401 to R407, R417 to R412, TP406 to TP400, TP405 to TP403
Changed lines of the file:
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@@
 		(on_board yes)
 		(dnp no)
-		(property "Reference" "TP405"
+		(property "Reference" "TP403"
 			(at 118.618 146.558 0)
 			(effects
@@
 			(project "Wireless_Charger"
 				(path "/547bfc24-3721-4bae-afe0-2e67b1f22193/ab5ffafb-c0a8-441f-b5fa-048ba9e5f69f"
-					(reference "TP405")
+					(reference "TP403")
 					(unit 1)
 				)
@@
 		(on_board yes)
 		(dnp no)
-		(property "Reference" "TP406"
+		(property "Reference" "TP400"
 			(at 119.38 93.218 0)
 			(effects
@@
 			(project "Wireless_Charger"
 				(path "/547bfc24-3721-4bae-afe0-2e67b1f22193/ab5ffafb-c0a8-441f-b5fa-048ba9e5f69f"
-					(reference "TP406")
+					(reference "TP400")
 					(unit 1)
 				)
@@
 		(on_board yes)
 		(dnp no)
-		(property "Reference" "R417"
+		(property "Reference" "R412"
 			(at 180.34 118.11 0)
 			(effects
@@
 			(project "Wireless_Charger"
 				(path "/547bfc24-3721-4bae-afe0-2e67b1f22193/ab5ffafb-c0a8-441f-b5fa-048ba9e5f69f"
-					(reference "R417")
+					(reference "R412")
 					(unit 1)
 				)
@@
 		(dnp no)
 		(fields_autoplaced yes)
-		(property "Reference" "R402"
+		(property "Reference" "R403"
 			(at 198.12 101.6 0)
 			(effects
@@
 			(project "Wireless_Charger"
 				(path "/547bfc24-3721-4bae-afe0-2e67b1f22193/ab5ffafb-c0a8-441f-b5fa-048ba9e5f69f"
-					(reference "R402")
+					(reference "R403")
 					(unit 1)
 				)
@@
 		(dnp no)
 		(fields_autoplaced yes)
-		(property "Reference" "R401"
+		(property "Reference" "R407"
 			(at 186.69 132.08 0)
 			(effects
@@
 			(project "Wireless_Charger"
 				(path "/547bfc24-3721-4bae-afe0-2e67b1f22193/ab5ffafb-c0a8-441f-b5fa-048ba9e5f69f"
-					(reference "R401")
+					(reference "R407")
 					(unit 1)
 				)
