File: Wireless_Charger.kicad_pcb (KiCad board)
At the start: 2 copper layers, 189 parts, among them J100 632723300011, J101 FTSH-107-01-L-DV-K-A, J201 0022232041, Q100 NTR4003NT1G, Q200 NTK3134NT1G, Q201 2N7002, Q202 2N7002, Q203 NTK3134NT1G, Q300 STL20N6F7, Q301 STL20N6F7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

Commit message: PCB Layout V1.1
Parts:
- removed R401, R402: 0R, Samacsys:RESC1005X40N
- removed R417: 10K, Samacsys:RESC1005X40N
- removed TP405, TP406: 1, TestPoint:TestPoint_Keystone_5015_Micro_Mini
- added R403: 0R, Samacsys:RESC1005X40N, F.Cu at (112.5, 119.4)
- added R407: 0R, Samacsys:RESC1005X40N, F.Cu at (112.5, 122.2)
- added R412: 10K, Samacsys:RESC1005X40N, F.Cu at (112.6, 117.9)
- added TP400: 1, TestPoint:TestPoint_Keystone_5015_Micro_Mini, F.Cu at (144.1, 105.4)
- added TP403: 1, TestPoint:TestPoint_Keystone_5015_Micro_Mini, F.Cu at (144.1, 132.7)
- moved C310 134.9 mm to (168.7, 150.2)
- moved C313 134.9 mm to (168.7, 152.9)
- moved C302 134.9 mm to (180.7, 144.5)
- moved Q300 134.9 mm to (169.7, 145.5)
- moved R303 134.9 mm to (165.2, 137.9)
- moved R305 134.9 mm to (210.9, 157.5)
- moved Q412 124.0 mm to (129.6, 149.1)
- moved Q411 123.7 mm to (134.7, 144.2)
- moved C402 109.9 mm to (134.9, 154.1)
- moved R423 107.4 mm to (129.9, 153.5)
- moved C423 106.6 mm to (134.9, 156.1), turned to 180 degrees
- moved R416 105.1 mm to (129.9, 155.1)
- moved R425 103.6 mm to (130.0, 151.9)
- moved R421 102.3 mm to (129.9, 156.6), turned to 180 degrees
- moved C425 99.9 mm to (134.9, 152.1), turned to 180 degrees
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Routing:
- net VIN: track 51.2 -> 0.00 mm, vias 6 -> 0
- net Net-(D102-D+-Pad1): track 0.00 -> 6.28 mm
- net Net-(J100-VBUS): track 0.00 -> 1.27 mm
- net VBRIDGE: vias 0 -> 24
- added copper zone on In1.Cu, net Earth
- added copper zone on F.Cu, net VBRIDGE
- added copper zone on In2.Cu, net VBRIDGE
Other:
- board outline added: 88.9 x 63.5 mm
- copper layers 2 -> 4

Commit message: Layout V1.2
Parts:
- D103: moved to B.Cu
- moved C221 176.0 mm to (60.1, 139.5), turned to 180 degrees
- moved C222 168.8 mm to (67.4, 139.5)
- moved D204 165.7 mm to (83.7, 136.3), turned to -90 degrees
- moved D205 165.1 mm to (82.3, 136.3), turned to -90 degrees
- moved D206 164.6 mm to (80.9, 136.3), turned to -90 degrees
- moved C236 164.3 mm to (79.5, 136.3), turned to -90 degrees
- moved C216 161.6 mm to (66.5, 135.1), turned to 180 degrees
- moved C238 157.5 mm to (59.3, 105.2), turned to -90 degrees
- moved C200 155.2 mm to (61.1, 123.4)
- moved C203 152.3 mm to (61.0, 121.6)
- moved D207 146.3 mm to (89.2, 120.3), turned to 180 degrees
- moved D208 143.0 mm to (89.3, 117.6), turned to 180 degrees
- moved CC230 141.8 mm to (94.4, 114.7), turned to 180 degrees
- moved C207 140.5 mm to (61.1, 105.2), turned to -90 degrees
- moved C237 139.9 mm to (101.7, 126.5)
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Connections:
- J100 pad B1: Earth -> VBUCK
- J100 pad B12: Earth -> VBUCK
- J201 pad 4: Earth -> VBUCK
Routing:
- net Net-(D102-D+-Pad1): track 6.28 -> 0.00 mm
- net Net-(J100-VBUS): track 1.27 -> 0.00 mm
- net VREF: vias 0 -> 3
- net VIN: vias 0 -> 15
- net VDD_DR: vias 0 -> 11
- net VDCDC: vias 0 -> 17
- net VBUCK: vias 0 -> 12
- net 3V3: vias 0 -> 13
- added copper zone on F.Cu, net 3V3
- added copper zone on In2.Cu, net 3V3
- added copper zone on F.Cu, net VBUCK
- added copper zone on In2.Cu, net VBUCK
- added copper zone on F.Cu, net VDCDC
- added copper zone on In2.Cu, net VDCDC
- added copper zone on F.Cu, net VDD_DR
- added copper zone on In2.Cu, net VDD_DR
- added copper zone on F.Cu, net VIN
- added copper zone on In2.Cu, net VIN
- added copper zone on F.Cu, net VREF
- added copper zone on In2.Cu, net VREF
Other:
- board size 88.9 x 63.5 mm -> 98.7 x 78.4 mm

Commit message: Layout V1.3
Parts:
- moved R307 28.9 mm to (63.7, 154.2)
- moved C315 28.8 mm to (65.2, 154.1), turned to 90 degrees
- moved R306 28.7 mm to (65.0, 156.1)
- moved R232 26.2 mm to (78.5, 101.3), turned to 0 degrees
- moved C241 21.5 mm to (75.8, 102.8), turned to -90 degrees
- moved R231 6.38 mm to (80.9, 100.7), turned to 0 degrees
- moved J100 3.87 mm to (51.3, 151.2)
- moved C215 2.36 mm to (81.1, 103.9)
- moved C240 2.36 mm to (78.5, 102.7)
- moved R230 2.36 mm to (78.5, 104.3)
- moved C214 2.36 mm to (81.9, 106.1)
- moved C218 2.36 mm to (81.2, 102.1)
- moved R204 2.36 mm to (79.1, 106.2)
- moved R229 2.36 mm to (77.9, 106.3)
Routing:
- net /SW_HS2: track 0.00 -> 55.7 mm
- net Net-(U203-IN-): track 0.00 -> 39.4 mm, vias 0 -> 2
- net Net-(C432-Pad2): track 0.00 -> 29.9 mm
- net /USB_D+: track 0.00 -> 28.5 mm, vias 0 -> 4
- net Net-(U200-BRG_FT_R): track 0.00 -> 24.1 mm
- net Net-(Q203-S): track 0.00 -> 24.0 mm, vias 0 -> 2
- net /BRIDGE_ISNS_N: track 0.00 -> 22.9 mm, vias 0 -> 2
- net Net-(U203-GND): track 0.00 -> 22.1 mm, vias 0 -> 2
- net Net-(L300-Pad2): track 0.00 -> 21.0 mm
- net /USB_D-: track 0.00 -> 20.4 mm
- net /I2C_SCL: track 0.00 -> 19.9 mm, vias 0 -> 2
- net /SW_HS1: track 0.00 -> 18.3 mm
- net /I2C_SDA: track 0.00 -> 18.0 mm
- net Net-(U200-BRG_IDEM): track 0.00 -> 17.0 mm
- net /RING_NODE2: track 0.00 -> 15.8 mm
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
Commit message: Layout V1.4
Routing:
- net VBUCK: track 0.00 -> 67.2 mm, vias 12 -> 15
- net /GD_LS1: track 0.00 -> 48.1 mm, vias 0 -> 4
- net /GD_LS3: track 0.00 -> 39.5 mm, vias 0 -> 2
- net /GD_HS1: track 0.00 -> 38.3 mm, vias 0 -> 2
- net /VIN_ISNS_N: track 1.93 -> 36.4 mm, vias 0 -> 2
- net /UART_TX: track 0.00 -> 26.5 mm
- net /QF_SHORT: track 0.00 -> 24.8 mm, vias 0 -> 2
- net Net-(U200-XTAL_OUT): track 2.68 -> 26.0 mm, vias 0 -> 2
- net /UART_RX: track 0.00 -> 23.1 mm
- net /TANK2_SEL: track 0.00 -> 22.6 mm, vias 0 -> 2
- net Net-(D103-I/O1): track 0.00 -> 21.6 mm, vias 0 -> 1
- net /SW_HS3: track 13.0 -> 31.8 mm, vias 0 -> 2
- net Net-(D103-I/O2): track 0.00 -> 16.7 mm, vias 0 -> 2
- net Net-(D204-K): track 1.41 -> 18.1 mm, vias 0 -> 2
- net 3V3: track 0.00 -> 14.2 mm, vias 13 -> 17
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
Commit message: Layout V1.5
Parts:
- moved TP403 7.21 mm to (144.2, 139.9)
- moved TP401 6.41 mm to (144.0, 105.3)
- moved TP400 6.14 mm to (144.0, 111.5)
- moved TP404 4.04 mm to (144.1, 135.0)
Routing:
- net VIN: track 0.00 -> 116.3 mm, vias 15 -> 18
- net /TANK1_SEL: track 0.00 -> 110.0 mm, vias 0 -> 4
- net /USB_DM: track 0.00 -> 86.6 mm, vias 0 -> 4
- net /USB_DP: track 0.00 -> 84.7 mm, vias 0 -> 4
- net VBUCK: track 67.2 -> 146.2 mm
- net /RING_NODE2: track 15.8 -> 90.3 mm, vias 0 -> 2
- net /BRIDGE_ISNS_N: track 22.9 -> 89.0 mm, vias 2 -> 4
- net /TANK2_SEL: track 22.6 -> 86.4 mm, vias 2 -> 4
- net /SWDIO: track 0.00 -> 63.1 mm, vias 0 -> 3
- net /SWCLK: track 0.00 -> 60.3 mm, vias 0 -> 3
- net /GD_HS3: track 0.00 -> 57.6 mm, vias 0 -> 4
- net /SW_HS3: track 31.8 -> 86.1 mm, vias 2 -> 6
- net VDD_DR: track 9.01 -> 62.0 mm
- net /RING_SNS: track 0.00 -> 49.5 mm, vias 0 -> 5
- net Net-(Q407-D): track 0.00 -> 48.7 mm, vias 0 -> 3
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- added copper zone on F.Cu, net Earth

Commit message: Layout V1.6
Parts:
- D103: moved to F.Cu
Routing:
- net Earth: track 8.46 -> 61.7 mm, vias 9 -> 98
- net Net-(U200-XTAL_IN): track 2.58 -> 31.6 mm, vias 0 -> 2
- net 3V3: track 50.6 -> 61.5 mm
- net VIN: track 116.3 -> 124.8 mm
- net Net-(Q403-G): track 0.00 -> 8.38 mm, vias 0 -> 2
- net Net-(Q401-G): track 0.00 -> 8.14 mm
- net VDCDC: track 49.0 -> 55.7 mm
- net Net-(C432-Pad2): track 29.9 -> 35.0 mm
- net Net-(Q402-G): track 0.00 -> 5.08 mm
- net Net-(D103-I/O2): track 16.7 -> 13.8 mm
- net /SW_HS1: track 54.2 -> 57.1 mm
- net VBUCK: track 146.2 -> 148.1 mm
- net Net-(U200-TEMPSNS): track 13.7 -> 14.4 mm
- net Net-(U200-BRG_VREF): track 13.7 -> 14.4 mm
- net Net-(U200-BUCK_BT): track 12.2 -> 13.0 mm
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
Commit message: Layout V1.7
Parts:
- moved TP200 0.08 mm to (50.4, 114.0)
Routing:
- net VBUCK: track 148.1 -> 154.1 mm, vias 15 -> 16
- net Net-(J100-VBUS): track 1.27 -> 5.40 mm
- net /USB_D+: track 28.5 -> 24.7 mm
- net Net-(Q203-S): track 24.0 -> 21.3 mm
- net /RING_NODE1: track 52.4 -> 54.3 mm
- net VDD_DR: track 62.0 -> 63.5 mm
- net Earth: track 61.7 -> 60.5 mm, vias 98 -> 96
- net /SWDIO: track 63.1 -> 62.0 mm
- net /GD_HS1: track 38.4 -> 39.4 mm
- net Net-(Q407-D): track 48.7 -> 49.5 mm
- net VDCDC: track 55.7 -> 56.5 mm
Other:
- board size 98.7 x 78.4 mm -> 98.7 x 60.1 mm
