File: usb_c.kicad_sch (KiCad schematic)
At the start: 22 parts, among them J100 632723300011, J101 FTSH-107-01-L-DV-K-A, Q100 NTR4003NT1G

Commit message: Layout V1.7
Connections:
- net USB_D+: now also J100.A7 (DN1), J100.B7 (DN2); no longer J100.A6 (DP1), J100.B6 (DP2)
- net USB_D-: now also J100.A6 (DP1), J100.B6 (DP2); no longer J100.A7 (DN1), J100.B7 (DN2)
- net VIN: now also J100.A5 (CC); no longer J100.B8 (SBU2)
- net at D103.2 (I/O2), R107.2: now also J100.B8 (SBU2); no longer J100.A5 (CC)
- net at J100.A8 (SBU1): now also D103.1 (I/O1), R106.1
- now unconnected: J100.B5 (VCONN)
Changed lines of the file:
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@@
 		(lib_id "CON_USB_C_632723300011:632723300011")
 		(at 83.82 63.5 0)
+		(mirror y)
 		(unit 1)
 		(exclude_from_sim no)
@@
 		(on_board yes)
 		(dnp no)
-		(fields_autoplaced yes)
 		(property "Reference" "J100"
 			(at 83.82 40.64 0)
